Commit message: changed parameters of model

File: scanner_description/urdf/scanner.xacro (robot description, xacro)
@@ -7,6 +7,6 @@
   <xacro:property name="width" value="0.1" /> <!-- Square dimensions (widthxwidth) of beams -->
   <xacro:property name="l0" value="${2 * axel_offset}" /> <!-- Link 1 -->
-  <xacro:property name="l1" value="1.5" /> <!-- Link 2 -->
-  <xacro:property name="l2" value="1.5" /> <!-- Link 3 -->
+  <xacro:property name="l1" value="1.55" /> <!-- Link 2 -->
+  <xacro:property name="l2" value="1.8" /> <!-- Link 3 -->
   <xacro:property name="h" value="${l0 + l1 + l2 + 2 * axel_offset}" /> <!-- Height of construction -->
   <xacro:property name="camera_link" value="0.05" /> <!-- Size of square 'camera' box -->

Commit message: camera pos fixed

File: scanner_description/urdf/scanner.xacro (robot description, xacro)
@@ -114,6 +114,6 @@
   </link>
   <joint name="camera_joint" type="fixed">
-    <axis xyz="0 1 0" />
-    <origin xyz="0 0 ${l2}" rpy="0 0 0"/>
+    <axis xyz="0 0 0" />
+    <origin xyz="0 0 ${l2 + width}" rpy="${-PI/2} ${-PI/2} ${-PI/2} "/>
     <parent link="link3"/>
     <child link="kinect_link"/>
@@ -123,5 +123,5 @@
       <origin xyz="0 0 0" rpy="0 0 0"/>
       <geometry>
-	<box size="0.1 0.1 0.1"/>
+	     <box size="0.1 0.1 0.1"/>
       </geometry>
     </collision>
@@ -176,61 +176,47 @@
     </actuator>
   </transmission>
-  <!-- <joint name="camera_joint" type="fixed">
-    <axis xyz="0 1 0" />
-    <origin xyz="${camera_link} 0 ${l2}" rpy="0 0 0"/>
-    <parent link="link3"/>
-    <child link="camera_link"/>
-  </joint> -->
-  <!-- Camera
-  <link name="camera_link">
-    <collision>
-      <origin xyz="0 0 0" rpy="0 0 0"/>
-      <geometry>
-	<box size="${camera_link} ${camera_link} ${camera_link}"/>
-      </geometry>
-    </collision>
-    <visual>
-      <origin xyz="0 0 0" rpy="0 0 0"/>
-      <geometry>
-	<box size="${camera_link} ${camera_link} ${camera_link}"/>
-      </geometry>
-      <material name="red"/>
-    </visual>
-    <inertial>
-      <mass value="1e-5" />
-      <origin xyz="0 0 0" rpy="0 0 0"/>
-      <inertia ixx="1e-6" ixy="0" ixz="0" iyy="1e-6" iyz="0" izz="1e-6" />
-    </inertial>
-  </link> -->
-  <!-- generate an optical frame http://www.ros.org/reps/rep-0103.html#suffix-frames
-      so that ros and opencv can operate on the camera frame correctly
-  <joint name="camera_optical_joint" type="fixed"> -->
-    <!-- these values have to be these values otherwise the gazebo camera image
-        won't be aligned properly with the frame it is supposedly originating from
-    <origin xyz="0 0 0" rpy="${-pi/2} 0 ${-pi/2}"/>
-    <parent link="camera_link"/>
-    <child link="camera_link_optical"/>
-  </joint>
-  <link name="camera_link_optical">
-  </link>-->
-  <!-- <transmission name="tran1">
-    <type>transmission_interface/SimpleTransmission</type>
-    <joint name="joint1">
-      <hardwareInterface>hardware_interface/EffortJointInterface</hardwareInterface>
-    </joint>
-    <actuator name="motor1">
-      <hardwareInterface>hardware_interface/EffortJointInterface</hardwareInterface>
-      <mechanicalReduction>1</mechanicalReduction>
-    </actuator>
-  </transmission>
-  <transmission name="tran2">
-    <type>transmission_interface/SimpleTransmission</type>
-    <joint name="joint2">
-      <hardwareInterface>hardware_interface/EffortJointInterface</hardwareInterface>
-    </joint>
-    <actuator name="motor2">
-      <hardwareInterface>hardware_interface/EffortJointInterface</hardwareInterface>
-      <mechanicalReduction>1</mechanicalReduction>
-    </actuator>
-  </transmission> -->
+  <!-- Here we go -->
+  <gazebo reference="kinect_link">
+    <sensor type="depth" name="camera1">
+        <always_on>1</always_on>
+        <visualize>true</visualize>
+        <camera>
+            <horizontal_fov>1.047</horizontal_fov>
+            <image>
+                <width>640</width>
+                <height>480</height>
+                <format>R8G8B8</format>
+            </image>
+            <depth_camera>
+            </depth_camera>
+            <clip>
+                <near>0.1</near>
+                <far>100</far>
+            </clip>
+        </camera>
+             <plugin name="camera_controller" filename="libgazebo_ros_openni_kinect.so">
+             <alwaysOn>true</alwaysOn>
+                <updateRate>1.0</updateRate>
+                <cameraName>camera</cameraName>
+                <frameName>kinect_link</frameName>
+            <imageTopicName>rgb/image_raw</imageTopicName>
+            <depthImageTopicName>depth/image_raw</depthImageTopicName>
+            <pointCloudTopicName>depth/points</pointCloudTopicName>
+            <cameraInfoTopicName>rgb/camera_info</cameraInfoTopicName>
+            <depthImageCameraInfoTopicName>depth/camera_info</depthImageCameraInfoTopicName>
+            <pointCloudCutoff>0.4</pointCloudCutoff>
+                <hackBaseline>0.07</hackBaseline>
+                <distortionK1>0.0</distortionK1>
+                <distortionK2>0.0</distortionK2>
+                <distortionK3>0.0</distortionK3>
+                <distortionT1>0.0</distortionT1>
+                <distortionT2>0.0</distortionT2>
+            <CxPrime>0.0</CxPrime>
+            <Cx>0.0</Cx>
+            <Cy>0.0</Cy>
+            <focalLength>0.0</focalLength>
+            </plugin>
+    </sensor>
+  </gazebo>
+  <!-- Here we finish -->
 </robot>

Commit message: Add Teleop, Configure Joints limitations

File: scanner_description/urdf/scanner.xacro (robot description, xacro)
@@ -9,5 +9,6 @@
   <xacro:property name="l1" value="1.55" /> <!-- Link 2 -->
   <xacro:property name="l2" value="1.8" /> <!-- Link 3 -->
-  <xacro:property name="h" value="${l0 + l1 + l2 + 2 * axel_offset}" /> <!-- Height of construction -->
+  <!-- Edit the last heigh as the axes is hitting the ground -->
+  <xacro:property name="h" value="${l0 + l1 + l2 + 4 * axel_offset}" /> <!-- (Height of construction -->
   <xacro:property name="camera_link" value="0.05" /> <!-- Size of square 'camera' box -->
   <xacro:property name="axel_offset" value="0.05" /> <!-- Space btw top of beam and the each joint -->
@@ -21,5 +22,6 @@
     <parent link="world"/>
     <child link="link1"/>
-    <origin xyz="0 0 ${h}" rpy="0 ${pi} 0"/>
+    <limit effort="1000.0" lower="0.0" upper="${PI*2}" velocity="0.5"/>
+    <origin xyz="0 0 ${h}" rpy="0 ${PI} 0"/>
     <axis xyz="0 0 1"/>
     <dynamics damping="0.7"/>
@@ -49,8 +51,8 @@
     </inertial>
   </link>
-  <joint name="joint1" type="continuous">
+  <joint name="joint1" type="revolute">
     <parent link="link1"/>
     <child link="link2"/>
-    <limit effort="1000.0" lower="0.0" upper="${pi/2}" velocity="0.5"/>
+    <limit effort="19000.0" lower="${-PI/2}" upper="${PI/2}" velocity="0.5"/>
     <origin xyz="0 ${width} ${l0}" rpy="0 0 0"/>
     <axis xyz="0 1 0"/>
@@ -81,8 +83,8 @@
     </inertial>
   </link>
-  <joint name="joint2" type="continuous">
+  <joint name="joint2" type="revolute">
     <parent link="link2"/>
     <child link="link3"/>
-    <limit effort="1000.0" lower="0" upper="${-pi}" velocity="0.5"/>
+    <limit effort="1000.0" lower="${-PI/2}" upper="${PI/2}" velocity="0.5"/>
     <origin xyz="0 ${width} ${l1}" rpy="0 0 0"/>
     <axis xyz="0 1 0"/>
@@ -100,5 +102,5 @@
       <origin xyz="0 0 ${l2/2}" rpy="0 0 0"/>
       <geometry>
-	<box size="${width} ${width} ${l2}"/>
+	      <box size="${width} ${width} ${l2}"/>
       </geometry>
       <material name="orange"/>
@@ -113,9 +115,10 @@
     </inertial>
   </link>
-  <joint name="camera_joint" type="fixed">
-    <axis xyz="0 0 0" />
-    <origin xyz="0 0 ${l2 + width}" rpy="${-PI/2} ${-PI/2} ${-PI/2} "/>
+  <joint name="camera_joint" type="revolute">
     <parent link="link3"/>
     <child link="kinect_link"/>
+    <limit effort="1000.0" lower="${-PI/2}" upper="${PI/2}" velocity="0.1"/>
+    <origin xyz="0 0 ${l2 + width}" rpy="${-PI/2} ${-PI/2} ${-PI/2} "/>
+    <axis xyz="0 1 0" />
   </joint>
   <link name="kinect_link">
@@ -126,4 +129,11 @@
       </geometry>
     </collision>
+    <!-- <collision name="collision">
+      <geometry>
+        <box>
+          <size>0.073000 0.276000 0.072000</size>
+        </box>
+      </geometry>
+    </collision> -->
     <visual>
       <origin xyz="0 0 0" rpy="0 0 0"/>
@@ -132,4 +142,12 @@
       </geometry>
     </visual>
+    <!-- <visual name="visual">
+      <origin xyz="0 0 0" rpy="0 0 0"/>
+        <geometry>
+          <mesh>
+            <uri>model://kinect/meshes/kinect.dae</uri>
+          </mesh>
+        </geometry>
+    </visual> -->
     <inertial>
       <mass value="1e-5" />
@@ -176,10 +194,34 @@
     </actuator>
   </transmission>
+  <transmission name="tran3">
+    <type>transmission_interface/SimpleTransmission</type>
+    <joint name="camera_joint">
+      <hardwareInterface>hardware_interface/EffortJointInterface</hardwareInterface>
+    </joint>
+    <actuator name="motor_kinect">
+      <hardwareInterface>hardware_interface/EffortJointInterface</hardwareInterface>
+      <mechanicalReduction>1</mechanicalReduction>
+    </actuator>
+  </transmission>
   <!-- Here we go -->
   <gazebo reference="kinect_link">
-    <sensor type="depth" name="camera1">
+    <!-- <sensor type="depth" name="camera1">
         <always_on>1</always_on>
-        <visualize>true</visualize>
-        <camera>
+        <visualize>true</visualize>              -->
+    <sensor name="camera" type="depth">
+      <update_rate>20</update_rate>
+      <camera>
+        <horizontal_fov>1.047198</horizontal_fov>
+        <image>
+          <width>640</width>
+          <height>480</height>
+          <format>R8G8B8</format>
+        </image>
+        <clip>
+          <near>0.05</near>
+          <far>3</far>
+        </clip>
+      </camera>
+        <!-- <camera>
             <horizontal_fov>1.047</horizontal_fov>
             <image>
@@ -194,29 +236,55 @@
                 <far>100</far>
             </clip>
-        </camera>
-             <plugin name="camera_controller" filename="libgazebo_ros_openni_kinect.so">
-             <alwaysOn>true</alwaysOn>
-                <updateRate>1.0</updateRate>
-                <cameraName>camera</cameraName>
-                <frameName>kinect_link</frameName>
-            <imageTopicName>rgb/image_raw</imageTopicName>
-            <depthImageTopicName>depth/image_raw</depthImageTopicName>
-            <pointCloudTopicName>depth/points</pointCloudTopicName>
-            <cameraInfoTopicName>rgb/camera_info</cameraInfoTopicName>
-            <depthImageCameraInfoTopicName>depth/camera_info</depthImageCameraInfoTopicName>
-            <pointCloudCutoff>0.4</pointCloudCutoff>
-                <hackBaseline>0.07</hackBaseline>
-                <distortionK1>0.0</distortionK1>
-                <distortionK2>0.0</distortionK2>
-                <distortionK3>0.0</distortionK3>
-                <distortionT1>0.0</distortionT1>
-                <distortionT2>0.0</distortionT2>
-            <CxPrime>0.0</CxPrime>
-            <Cx>0.0</Cx>
-            <Cy>0.0</Cy>
-            <focalLength>0.0</focalLength>
-            </plugin>
+        </camera> -->
+        <plugin name="camera_controller" filename="libgazebo_ros_openni_kinect.so">
+          <alwaysOn>true</alwaysOn>
+          <updateRate>1.0</updateRate>
+          <cameraName>camera</cameraName>
+          <frameName>kinect_link</frameName>
+          <imageTopicName>rgb/image_raw</imageTopicName>
+          <depthImageTopicName>depth/image_raw</depthImageTopicName>
+          <pointCloudTopicName>depth/points</pointCloudTopicName>
+          <cameraInfoTopicName>rgb/camera_info</cameraInfoTopicName>
+          <depthImageCameraInfoTopicName>depth/camera_info</depthImageCameraInfoTopicName>
+          <pointCloudCutoff>0.4</pointCloudCutoff>
+          <hackBaseline>0.07</hackBaseline>
+          <distortionK1>0.0</distortionK1>
+          <distortionK2>0.0</distortionK2>
+          <distortionK3>0.0</distortionK3>
+          <distortionT1>0.0</distortionT1>
+          <distortionT2>0.0</distortionT2>
+          <CxPrime>0.0</CxPrime>
+          <Cx>0.0</Cx>
+          <Cy>0.0</Cy>
+          <focalLength>0.0</focalLength>
+        </plugin>
     </sensor>
   </gazebo>
+<!-- <pose>0 0 0.036 0 0 0</pose>
+        <plugin name="camera_plugin" filename="libgazebo_ros_openni_kinect.so">
+          <baseline>0.2</baseline>
+          <alwaysOn>true</alwaysOn>
+          <updateRate>0.0</updateRate>
+          <cameraName>camera_ir</cameraName>
+          <imageTopicName>/camera/depth/image_raw</imageTopicName>
+          <cameraInfoTopicName>/camera/depth/camera_info</cameraInfoTopicName>
+          <depthImageTopicName>/camera/depth/image_raw</depthImageTopicName>
+          <depthImageInfoTopicName>/camera/depth/camera_info</depthImageInfoTopicName>
+          <pointCloudTopicName>/camera/depth/points</pointCloudTopicName>
+          <frameName>camera_link</frameName>
+          <pointCloudCutoff>0.05</pointCloudCutoff>
+          <distortionK1>0</distortionK1>
+          <distortionK2>0</distortionK2>
+          <distortionK3>0</distortionK3>
+          <distortionT1>0</distortionT1>
+          <distortionT2>0</distortionT2>
+          <CxPrime>0</CxPrime>
+          <Cx>0</Cx>
+          <Cy>0</Cy>
+          <focalLength>0</focalLength>
+          <hackBaseline>0</hackBaseline>
+        </plugin>
+      </sensor>
+    </link> -->
   <!-- Here we finish -->
 </robot>

Commit message: Rotate the kinect successfully

File: scanner_description/urdf/scanner.xacro (robot description, xacro)
@@ -115,10 +115,11 @@
     </inertial>
   </link>
-  <joint name="camera_joint" type="revolute">
+  <joint name="kinect_joint" type="revolute">
     <parent link="link3"/>
     <child link="kinect_link"/>
-    <limit effort="1000.0" lower="${-PI/2}" upper="${PI/2}" velocity="0.1"/>
+    <limit effort="1000.0" lower="${-PI/2}" upper="${PI/2}" velocity="0.5"/>
+    <axis xyz="0 0 1" />
     <origin xyz="0 0 ${l2 + width}" rpy="${-PI/2} ${-PI/2} ${-PI/2} "/>
-    <axis xyz="0 1 0" />
+    <dynamics damping="0.7"/>
   </joint>
   <link name="kinect_link">
@@ -129,11 +130,4 @@
       </geometry>
     </collision>
-    <!-- <collision name="collision">
-      <geometry>
-        <box>
-          <size>0.073000 0.276000 0.072000</size>
-        </box>
-      </geometry>
-    </collision> -->
     <visual>
       <origin xyz="0 0 0" rpy="0 0 0"/>
@@ -142,17 +136,13 @@
       </geometry>
     </visual>
-    <!-- <visual name="visual">
+    <inertial>
+      <!-- <mass value="1e-5" /> -->
       <origin xyz="0 0 0" rpy="0 0 0"/>
-        <geometry>
-          <mesh>
-            <uri>model://kinect/meshes/kinect.dae</uri>
-          </mesh>
-        </geometry>
-    </visual> -->
-    <inertial>
-      <mass value="1e-5" />
-      <origin xyz="0 0 0" rpy="0 0 0"/>
-      <inertia ixx="1e-6" ixy="0" ixz="0" iyy="1e-6" iyz="0" izz="1e-6" />
-    </inertial>
+      <mass value="${mass}"/>
+      <inertia
+        ixx="${mass * (0.1*0.1 + 0.1*0.1)}" ixy="0.0" ixz="0.0"
+        iyy="${mass * (0.1*0.1 + 0.1*0.1)}" iyz="0.0"
+        izz="${mass * (0.1*0.1 + 0.1*0.1)}"/>
+      </inertial>
   </link>
   <!--                GAZEBO RELATED PART                             -->
@@ -196,8 +186,8 @@
   <transmission name="tran3">
     <type>transmission_interface/SimpleTransmission</type>
-    <joint name="camera_joint">
-      <hardwareInterface>hardware_interface/EffortJointInterface</hardwareInterface>
-    </joint>
-    <actuator name="motor_kinect">
+    <joint name="kinect_joint">
+      <hardwareInterface>hardware_interface/EffortJointInterface</hardwareInterface>
+    </joint>
+    <actuator name="motor3">
       <hardwareInterface>hardware_interface/EffortJointInterface</hardwareInterface>
       <mechanicalReduction>1</mechanicalReduction>

Commit message: modified world and model. fixed camera

File: scanner_description/urdf/scanner.xacro (robot description, xacro)
@@ -10,5 +10,5 @@
   <xacro:property name="l2" value="1.8" /> <!-- Link 3 -->
   <!-- Edit the last heigh as the axes is hitting the ground -->
-  <xacro:property name="h" value="${l0 + l1 + l2 + 4 * axel_offset}" /> <!-- (Height of construction -->
+  <xacro:property name="h" value="${l0 + l2 + 10 * axel_offset}" /> <!-- (Height of construction -->
   <xacro:property name="camera_link" value="0.05" /> <!-- Size of square 'camera' box -->
   <xacro:property name="axel_offset" value="0.05" /> <!-- Space btw top of beam and the each joint -->
@@ -22,5 +22,5 @@
     <parent link="world"/>
     <child link="link1"/>
-    <limit effort="1000.0" lower="0.0" upper="${PI*2}" velocity="0.5"/>
+    <limit effort="1000.0"  velocity="0.5"/>
     <origin xyz="0 0 ${h}" rpy="0 ${PI} 0"/>
     <axis xyz="0 0 1"/>
@@ -51,9 +51,9 @@
     </inertial>
   </link>
-  <joint name="joint1" type="revolute">
+  <joint name="joint1" type="fixed">
     <parent link="link1"/>
     <child link="link2"/>
     <limit effort="19000.0" lower="${-PI/2}" upper="${PI/2}" velocity="0.5"/>
-    <origin xyz="0 ${width} ${l0}" rpy="0 0 0"/>
+    <origin xyz="0 ${width} ${l0}" rpy="0 ${PI/2} 0"/>
     <axis xyz="0 1 0"/>
     <dynamics damping="0.7"/>
@@ -83,9 +83,9 @@
     </inertial>
   </link>
-  <joint name="joint2" type="revolute">
+  <joint name="joint2" type="fixed">
     <parent link="link2"/>
     <child link="link3"/>
     <limit effort="1000.0" lower="${-PI/2}" upper="${PI/2}" velocity="0.5"/>
-    <origin xyz="0 ${width} ${l1}" rpy="0 0 0"/>
+    <origin xyz="0 ${width} ${l1}" rpy="0 ${-PI/2} 0"/>
     <axis xyz="0 1 0"/>
     <dynamics damping="0.7"/>
@@ -115,10 +115,33 @@
     </inertial>
   </link>
-  <joint name="kinect_joint" type="revolute">
+  <link name="link4">
+    <collision>
+      <origin xyz="0 0 ${width/2}" rpy="0 0 0"/>
+      <geometry>
+  <box size="${width} ${width} ${width}"/>
+      </geometry>
+    </collision>
+    <visual>
+      <origin xyz="0 0 ${width/2}" rpy="0 0 0"/>
+      <geometry>
+        <box size="${width} ${width} ${width}"/>
+      </geometry>
+      <material name="orange"/>
+    </visual>
+    <inertial>
+      <origin xyz="0 0 ${width/2}" rpy="0 0 0"/>
+      <mass value="${mass}"/>
+      <inertia
+    ixx="${mass / 12.0 * (width*width + width*width)}" ixy="0.0" ixz="0.0"
+    iyy="${mass / 12.0 * (width*width + width*width)}" iyz="0.0"
+    izz="${mass / 12.0 * (width*width + width*width)}"/>
+    </inertial>
+  </link>
+   <joint name="l3_to_l4_joint" type="fixed">
     <parent link="link3"/>
-    <child link="kinect_link"/>
+    <child link="link4"/>
     <limit effort="1000.0" lower="${-PI/2}" upper="${PI/2}" velocity="0.5"/>
     <axis xyz="0 0 1" />
-    <origin xyz="0 0 ${l2 + width}" rpy="${-PI/2} ${-PI/2} ${-PI/2} "/>
+    <origin xyz="0 0 ${l2}" rpy="0 ${-PI/2} 0"/>
     <dynamics damping="0.7"/>
   </joint>
@@ -127,5 +150,5 @@
       <origin xyz="0 0 0" rpy="0 0 0"/>
       <geometry>
-	     <box size="0.1 0.1 0.1"/>
+	     <box size="0.1 0.05 0.01"/>
       </geometry>
     </collision>
@@ -133,5 +156,5 @@
       <origin xyz="0 0 0" rpy="0 0 0"/>
       <geometry>
-       <box size="0.1 0.1 0.1"/>
+       <box size="0.1 0.05 0.01"/>
       </geometry>
     </visual>
@@ -146,4 +169,18 @@
       </inertial>
   </link>
+  <joint name="kinect_joint" type="fixed">
+    <parent link="link4"/>
+    <child link="kinect_link"/>
+    <limit effort="1000.0" lower="${-PI/2}" upper="${PI/2}" velocity="0.5"/>
+    <axis xyz="0 0 1" />
+    <origin xyz="0 0 ${width}" rpy="${-PI/2} ${-PI/2} ${PI/2} "/>
+    <dynamics damping="0.7"/>
+  </joint>
+  <joint name="cameraLeft_depth_joint" type="fixed">
+    <origin xyz="0 0 0" rpy="${-PI/2} 0 ${-PI/2} "/>
+    <parent link="kinect_link"/>
+    <child link="cameraLeft_depth_link"/>
+  </joint>
+  <link name="cameraLeft_depth_link"></link>
   <!--                GAZEBO RELATED PART                             -->
   <!-- ROS Control plugin for Gazebo -->
@@ -164,4 +201,5 @@
     </actuator>
   </transmission>
+<!--
   <transmission name="tran1">
     <type>transmission_interface/SimpleTransmission</type>
@@ -193,5 +231,5 @@
       <mechanicalReduction>1</mechanicalReduction>
     </actuator>
-  </transmission>
+  </transmission> -->
   <!-- Here we go -->
   <gazebo reference="kinect_link">
@@ -231,5 +269,5 @@
           <updateRate>1.0</updateRate>
           <cameraName>camera</cameraName>
-          <frameName>kinect_link</frameName>
+          <frameName>cameraLeft_depth_link</frameName>
           <imageTopicName>rgb/image_raw</imageTopicName>
           <depthImageTopicName>depth/image_raw</depthImageTopicName>

Commit message: configs changed. not for master

File: scanner_description/urdf/scanner.xacro (robot description, xacro)
@@ -10,5 +10,5 @@
   <xacro:property name="l2" value="1.8" /> <!-- Link 3 -->
   <!-- Edit the last heigh as the axes is hitting the ground -->
-  <xacro:property name="h" value="${l0 + l2 + 10 * axel_offset}" /> <!-- (Height of construction -->
+  <xacro:property name="h" value="${l0 + l2 + 7 * axel_offset}" /> <!-- (Height of construction -->
   <xacro:property name="camera_link" value="0.05" /> <!-- Size of square 'camera' box -->
   <xacro:property name="axel_offset" value="0.05" /> <!-- Space btw top of beam and the each joint -->
@@ -87,5 +87,5 @@
     <child link="link3"/>
     <limit effort="1000.0" lower="${-PI/2}" upper="${PI/2}" velocity="0.5"/>
-    <origin xyz="0 ${width} ${l1}" rpy="0 ${-PI/2} 0"/>
+    <origin xyz="0 ${-width} ${l1}" rpy="0 ${-PI/2} 0"/>
     <axis xyz="0 1 0"/>
     <dynamics damping="0.7"/>
